File: projekt/projekt-backups/projekt-2025-11-04_101825/projekt.kicad_sch (KiCad schematic)
At the start: 47 parts, among them J1 Conn_01x02, SW1 SW_Nidec_CAS-120A1, SW2 SW_Push, U1 LM2574N-5, U2 4027, U3 4027, U5 NE555P, U6 74LS47, U7 HDSP-7501, U8 4027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

Commit message: 25.11.
25.11.
Parts:
- renumbered 4k7 to 4k1, 4k7 to 4k2, 4k7 to 4k3, C5 to C1, C3 to C2, C1 to C3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
